File: tproject.kicad_pcb (KiCad board)
At the start: 2 copper layers, 38.5 x 33.2 mm, 32 parts, among them J1 USB_B_Micro, J2 Conn_01x04_Pin, J3 Conn_01x04_Pin, J4 Conn_01x04_Pin, SW1 SW_SPDT, U1 STM32F103C8T6, U2 AMS1117-3.3, Y1 16MHz

Commit message: power-routing
Parts:
- moved U2 3.56 mm to (64.2, 76.2)
- moved R1 3.47 mm to (73.0, 72.0), turned to 0 degrees
- moved C2 2.36 mm to (69.0, 75.7)
- moved D1 1.97 mm to (72.5, 75.8), turned to -90 degrees
- moved C1 1.68 mm to (64.3, 70.5)
Routing:
- net +3.3V: track 7.79 -> 145.8 mm, vias 0 -> 4
- net GND: track 9.80 -> 33.4 mm, vias 0 -> 17
- net /NRST: track 0.00 -> 9.50 mm
- net +3.3VA: track 2.18 -> 7.46 mm
- net /PWR_LED_K: track 0.00 -> 3.01 mm
- net (no net): track 0.00 -> 0.83 mm, vias 0 -> 6
- added copper zone on F.Cu, net +3.3V
- added copper zone on F.Cu, net GND
- added copper zone on F.Cu, net VBUS

Commit message: the end of the course
Other:
- board text added: "1.0.0"
- board text added: "3May26"
- board text added: "BOOT"
- board text added: "I2C"
- board text added: "ON"
- board text added: "SWD"
- board text added: "UART"
- board text added: "USB"
- board text added: "itma.tech"
Changed lines of the file:
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@@
 			(outputformat 1)
 			(mirror no)
-			(drillshape 1)
+			(drillshape 0)
 			(scaleselection 1)
-			(outputdirectory "")
+			(outputdirectory "manufacturing/")
 		)
 	)
@@
 		(tags "Through hole pin header THT 1x04 2.54mm single row")
 		(property "Reference" "J4"
-			(at 0 -2.38 90)
+			(at -0.5 -2.67 180)
 			(layer "F.SilkS")
 			(effects
@@
 		(layer "Edge.Cuts")
 	)
+	(gr_text "BOOT"
+		(at 37.5 70.5 0)
+		(layer "F.SilkS")
+		(effects
+			(font
+				(size 1 1)
+				(thickness 0.1)
+			)
+			(justify left bottom)
+		)
+	)
+	(gr_text "UART"
+		(at 45 53.5 0)
+		(layer "F.SilkS")
+		(effects
+			(font
+				(size 1 1)
+				(thickness 0.1)
+			)
+			(justify left bottom)
+		)
+	)
+	(gr_text "I2C"
+		(at 46.5 81.5 0)
+		(layer "F.SilkS")
+		(effects
+			(font
+				(size 1 1)
+				(thickness 0.1)
+			)
+			(justify left bottom)
+		)
+	)
+	(gr_text "USB"
+		(at 70.75 60.25 0)
+		(layer "F.SilkS")
+		(effects
+			(font
+				(size 1 1)
+				(thickness 0.1)
+			)
+			(justify left bottom)
+		)
+	)
+	(gr_text "ON"
+		(at 72.25 78.25 0)
+		(layer "F.SilkS")
+		(effects
+			(font
+				(size 1 1)
+				(thickness 0.1)
+			)
+			(justify left bottom)
+		)
+	)
+	(gr_text "SWD"
+		(at 59.75 53.5 0)
+		(layer "F.SilkS")
+		(effects
+			(font
+				(size 1 1.25)
+				(thickness 0.1)
+			)
+			(justify left bottom)
+		)
+	)
+	(gr_text "1.0.0"
+		(at 42 75.25 0)
+		(layer "B.SilkS")
+		(effects
+			(font
+				(size 1 1)
+				(thickness 0.1)
+			)
+			(justify left bottom mirror)
+		)
+	)
+	(gr_text "3May26"
+		(at 43.5 77.25 0)
+		(layer "B.SilkS")
+		(effects
+			(font
+				(size 1 1)
+				(thickness 0.1)
+			)
+			(justify left bottom mirror)
+		)
+	)
+	(gr_text "itma.tech"
+		(at 44 79 0)
+		(layer "B.SilkS")
+		(effects
+			(font
+				(size 1 1)
+				(thickness 0.1)
+			)
+			(justify left bottom mirror)
+		)
+	)
 	(segment
 		(start 67 64.75)
@@
 		(min_thickness 0.25)
 		(filled_areas_thickness no)
-		(fill
+		(fill yes
 			(thermal_gap 0.5)
 			(thermal_bridge_width 0.5)
@@
 		(min_thickness 0.25)
 		(filled_areas_thickness no)
-		(fill
+		(fill yes
 			(thermal_gap 0.5)
 			(thermal_bridge_width 0.5)
@@
 		(min_thickness 0.25)
 		(filled_areas_thickness no)
-		(fill
+		(fill yes
 			(thermal_gap 0.5)
 			(thermal_bridge_width 0.5)
